File: RocketHat.kicad_pcb (KiCad board)
At the start: 2 copper layers, 72.2 x 58.1 mm, 28 parts, among them J1 Conn_01x06_Female, J10 Conn_01x10_Female, J11 Raspberry_Pi_2_3, J2 Conn_01x06_Female, J3 Conn_01x07_Female, J4 Conn_01x06_Female, J5 Conn_01x04_Female, J6 Conn_01x02_Female, J7 Conn_01x02, J8 Conn_01x10_Female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

Commit message: Version 1.1.0
Parts:
- removed J11: Raspberry_Pi_2_3, Connector_PinSocket_2.54mm:PinSocket_2x20_P2.54mm_Vertical
- removed JP1: SolderJumper_2_Open, Jumper:SolderJumper-2_P1.3mm_Open_TrianglePad1.0x1.5mm
- removed Q2: DMG2305UX-13, digikey-footprints:SOT-23-3
- removed Q3: 2N3904, Package_TO_SOT_THT:TO-92_Inline
- removed R1: 10K, Resistor_SMD:R_0603_1608Metric
- removed R6: 3.9K, Resistor_SMD:R_0603_1608Metric
- added JP2: SolderJumper_2_Open, Jumper:SolderJumper-2_P1.3mm_Open_TrianglePad1.0x1.5mm, F.Cu at (111.8, 76.3)
- J1: value Conn_01x06_Female -> Screw_Terminal_01x02; footprint Connector_PinSocket_2.54mm:PinSocket_1x06_P2.54mm_Vertical -> TerminalBlock_Phoenix:TerminalBlock_Phoenix_MKDS-1,5-2_1x02_P5.00mm_Horizontal
- J10: value Conn_01x10_Female -> Raspberry_Pi_2_3; footprint Connector_PinSocket_2.00mm:PinSocket_1x10_P2.00mm_Vertical -> Connector_PinSocket_2.54mm:PinSocket_2x20_P2.54mm_Vertical
- J3: value Conn_01x07_Female -> Conn_01x06_Female; footprint Connector_PinSocket_2.54mm:PinSocket_1x07_P2.54mm_Vertical -> Connector_PinSocket_2.54mm:PinSocket_1x06_P2.54mm_Vertical
- J4: value Conn_01x06_Female -> Conn_01x07_Female; footprint Connector_PinSocket_2.54mm:PinSocket_1x06_P2.54mm_Vertical -> Connector_PinSocket_2.54mm:PinSocket_1x07_P2.54mm_Vertical
- J5: value Conn_01x04_Female -> Conn_01x06_Female; footprint Connector_PinSocket_2.54mm:PinSocket_1x04_P2.54mm_Vertical -> Connector_PinSocket_2.54mm:PinSocket_1x06_P2.54mm_Vertical
- J6: value Conn_01x02_Female -> Conn_01x04_Female; footprint Connector_Wago:Wago_734-162_1x02_P3.50mm_Horizontal -> Connector_PinSocket_2.54mm:PinSocket_1x04_P2.54mm_Vertical
- J7, J9: value Conn_01x02 -> Conn_01x10_Female; footprint Connector_PinHeader_2.54mm:PinHeader_1x02_P2.54mm_Vertical -> Connector_PinSocket_2.00mm:PinSocket_1x10_P2.00mm_Vertical
- J8: value Conn_01x10_Female -> Conn_01x02; footprint Connector_PinSocket_2.00mm:PinSocket_1x10_P2.00mm_Vertical -> Connector_PinHeader_2.54mm:PinHeader_1x02_P2.54mm_Vertical
- Q1: value 2N3904 -> FQP27P06; footprint Package_TO_SOT_THT:TO-92_Inline -> Package_TO_SOT_THT:TO-220-3_Vertical
- R2: value 47K -> 10K; footprint Resistor_SMD:R_0603_1608Metric -> Resistor_THT:R_Axial_DIN0204_L3.6mm_D1.6mm_P5.08mm_Horizontal
- R3: value 10K -> 10K 1%; footprint Resistor_SMD:R_0603_1608Metric -> Resistor_THT:R_Axial_DIN0204_L3.6mm_D1.6mm_P5.08mm_Horizontal
- R4: value 10K 1% -> 3.9K; footprint Resistor_SMD:R_0603_1608Metric -> Resistor_THT:R_Axial_DIN0204_L3.6mm_D1.6mm_P5.08mm_Horizontal; moved to F.Cu
- R5: footprint Resistor_SMD:R_0603_1608Metric -> Resistor_THT:R_Axial_DIN0204_L3.6mm_D1.6mm_P5.08mm_Horizontal; moved to F.Cu
- U1: moved to F.Cu
- moved J1 86.3 mm to (87.9, 65.0)
- moved H6 85.9 mm to (93.1, 79.2)
- moved J9 67.7 mm to (93.5, 36.9), turned to 90 degrees
- moved J5 50.1 mm to (133.6, 65.0), turned to 90 degrees
- moved J2 48.2 mm to (133.6, 82.8), turned to 90 degrees
- moved J10 37.8 mm to (98.0, 28.9)
- moved J4 36.7 mm to (150.1, 52.5), turned to 180 degrees
- moved Q1 36.3 mm to (97.6, 70.1), turned to 90 degrees
- moved H2 34.9 mm to (132.5, 51.0)
- moved H1 33.5 mm to (132.4, 38.6)
- moved R3 32.2 mm to (137.8, 42.3), turned to 90 degrees
- moved H3 30.5 mm to (151.1, 79.2)
- moved J3 28.9 mm to (108.1, 83.5), turned to 90 degrees
- moved H4 27.9 mm to (151.1, 30.2)
- moved H5 27.7 mm to (93.1, 30.3)
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Connections:
- J1 pad 1: /3V3 -> Net-(J1-Pad1)
- J1 pad 2: unconnected-(J1-Pad2) -> GND
- J10 pad 1: unconnected-(J10-Pad1) -> /3V3
- J10 pad 10: unconnected-(J10-Pad10) -> /XBEE_TX
- J10 pad 2: unconnected-(J10-Pad2) -> /P5V_HAT
- J10 pad 4: unconnected-(J10-Pad4) -> /P5V_HAT
- J10 pad 6: unconnected-(J10-Pad6) -> GND
- J10 pad 8: unconnected-(J10-Pad8) -> /XBEE_RX
- J10 pad 9: unconnected-(J10-Pad9) -> GND
- J3 pad 2: GND -> unconnected-(J3-Pad2)
- J3 pad 3: unconnected-(J3-Pad3) -> GND
- J3 pad 4: unconnected-(J3-Pad4) -> /SENSOR_SCL
- J3 pad 5: unconnected-(J3-Pad5) -> /SENSOR_SDA
- J3 pad 6: /SENSOR_SCL -> unconnected-(J3-Pad6)
- J4 pad 1: unconnected-(J4-Pad1) -> /3V3
- J4 pad 2: unconnected-(J4-Pad2) -> GND
- J4 pad 6: unconnected-(J4-Pad6) -> /SENSOR_SCL
- J5 pad 2: /ADR_BNO055 -> unconnected-(J5-Pad2)
- J6 pad 1: /P5V -> unconnected-(J6-Pad1)
- J6 pad 2: GND -> /ADR_BNO055
- J7 pad 1: /P5V_HAT -> /3V3
- J7 pad 2: /P5V -> /XBEE_TX
- J8 pad 1: /3V3 -> Net-(J8-Pad1)
- J8 pad 2: /XBEE_TX -> GND
- J9 pad 1: Net-(J9-Pad1) -> unconnected-(J9-Pad1)
- J9 pad 2: GND -> unconnected-(J9-Pad2)
- Q1 pad 1: /P5V -> GND
- Q1 pad 2: Net-(Q1-Pad2) -> Net-(J1-Pad1)
- Q1 pad 3: Net-(Q1-Pad2) -> /P5V_HAT
- R2 pad 1: Net-(Q2-Pad1) -> /ADR_BNO055
- R3 pad 1: /ADR_BNO055 -> Net-(J8-Pad1)
- R3 pad 2: GND -> /3V3
- R4 pad 1: Net-(J9-Pad1) -> /3V3
- R4 pad 2: /3V3 -> /EEPROM_SDA
- R5 pad 2: /EEPROM_SDA -> /EEPROM_SCL
- U1 pad 7: Net-(J9-Pad1) -> Net-(J8-Pad1)
Routing:
- net GND: track 179.6 -> 10.7 mm
- net /P5V: track 49.0 -> 0.00 mm
- net /3V3: track 162.0 -> 198.9 mm
- net /SENSOR_SDA: track 75.8 -> 110.6 mm, vias 1 -> 0
- net /SENSOR_SCL: track 81.6 -> 113.7 mm
- net Net-(J8-Pad1): track 0.00 -> 26.5 mm
- net Net-(Q1-Pad2): track 24.0 -> 0.00 mm
- net Net-(J9-Pad1): track 22.8 -> 0.00 mm
- net Net-(Q2-Pad1): track 19.2 -> 0.00 mm
- net /P5V_HAT: track 30.3 -> 45.0 mm
- net Net-(J1-Pad1): track 0.00 -> 10.7 mm
- net /EEPROM_SDA: track 17.2 -> 26.3 mm
- net /ADR_BNO055: track 22.9 -> 14.4 mm
- net /XBEE_TX: track 31.1 -> 37.6 mm
- net /XBEE_RX: track 32.1 -> 30.8 mm
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Other:
- board size 72.2 x 58.1 mm -> 72.2 x 60.3 mm
- board text added: "Made With Love <3"
- board text added: "Version 1.1"
- board text removed: "+"
- board text removed: "-"
- board text removed: "HI MOMS"
- board text removed: "Version 1.0"

Commit message: Added Graphic
Parts:
- added G***: LOGO, RocketLogo:rocketry-logo, B.Cu at (87.1, 44.2)
Routing:
- net /3V3: track 198.9 -> 250.4 mm
Other:
- board text added: "X ->"

Commit message: PCB Updates
Connections:
- J10 pad 15: unconnected-(J10-Pad15) -> /BNORST
- J3 pad 6: unconnected-(J3-Pad6) -> /BNORST
Changed lines of the file:
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@@
   (net 10 "/XBEE_TX")
   (net 11 "unconnected-(J3-Pad2)")
-  (net 12 "unconnected-(J3-Pad6)")
+  (net 12 "/BNORST")
   (net 13 "unconnected-(J5-Pad2)")
   (net 14 "unconnected-(J5-Pad5)")
@@
   (net 48 "unconnected-(J5-Pad4)")
   (net 49 "unconnected-(J10-Pad13)")
-  (net 50 "unconnected-(J10-Pad15)")
-  (net 51 "unconnected-(J10-Pad16)")
-  (net 52 "unconnected-(J10-Pad18)")
-  (net 53 "unconnected-(J10-Pad19)")
-  (net 54 "unconnected-(J10-Pad21)")
-  (net 55 "unconnected-(J10-Pad22)")
-  (net 56 "unconnected-(J10-Pad26)")
-  (net 57 "unconnected-(J10-Pad29)")
-  (net 58 "unconnected-(J10-Pad31)")
-  (net 59 "unconnected-(J10-Pad32)")
-  (net 60 "unconnected-(J10-Pad33)")
-  (net 61 "unconnected-(J10-Pad35)")
-  (net 62 "unconnected-(J10-Pad36)")
-  (net 63 "unconnected-(J10-Pad37)")
-  (net 64 "unconnected-(J10-Pad38)")
-  (net 65 "unconnected-(J10-Pad40)")
+  (net 50 "unconnected-(J10-Pad16)")
+  (net 51 "unconnected-(J10-Pad18)")
+  (net 52 "unconnected-(J10-Pad19)")
+  (net 53 "unconnected-(J10-Pad21)")
+  (net 54 "unconnected-(J10-Pad22)")
+  (net 55 "unconnected-(J10-Pad26)")
+  (net 56 "unconnected-(J10-Pad29)")
+  (net 57 "unconnected-(J10-Pad31)")
+  (net 58 "unconnected-(J10-Pad32)")
+  (net 59 "unconnected-(J10-Pad33)")
+  (net 60 "unconnected-(J10-Pad35)")
+  (net 61 "unconnected-(J10-Pad36)")
+  (net 62 "unconnected-(J10-Pad37)")
+  (net 63 "unconnected-(J10-Pad38)")
+  (net 64 "unconnected-(J10-Pad40)")
   (footprint "Resistor_THT:R_Axial_DIN0204_L3.6mm_D1.6mm_P5.08mm_Horizontal" (layer "F.Cu")
     (at 137.778 42.2954 90)
@@
       (net 6 "/SENSOR_SDA") (pinfunction "Pin_5") (pintype "passive"))
     (pad "6" thru_hole oval locked (at 0 12.7 90) (size 1.7 1.7) (drill 1) (layers *.Cu *.Mask)
-      (net 12 "unconnected-(J3-Pad6)") (pinfunction "Pin_6") (pintype "passive+no_connect"))
+      (net 12 "/BNORST") (pinfunction "Pin_6") (pintype "passive"))
     (model "${KICAD6_3DMODEL_DIR}/Connector_PinSocket_2.54mm.3dshapes/PinSocket_1x06_P2.54mm_Vertical.wrl"
       (offset (xyz 0 0 0))
@@
       (net 2 "GND") (pinfunction "GND") (pintype "power_in"))
     (pad "15" thru_hole oval locked (at 0 17.78 90) (size 1.7 1.7) (drill 1) (layers *.Cu *.Mask)
-      (net 50 "unconnected-(J10-Pad15)") (pinfunction "GPIO22") (pintype "bidirectional+no_connect"))
+      (net 12 "/BNORST") (pinfunction "GPIO22") (pintype "bidirectional"))
     (pad "16" thru_hole oval locked (at -2.54 17.78 90) (size 1.7 1.7) (drill 1) (layers *.Cu *.Mask)
-      (net 51 "unconnected-(J10-Pad16)") (pinfunction "GPIO23") (pintype "bidirectional+no_connect"))
+      (net 50 "unconnected-(J10-Pad16)") (pinfunction "GPIO23") (pintype "bidirectional+no_connect"))
     (pad "17" thru_hole oval locked (at 0 20.32 90) (size 1.7 1.7) (drill 1) (layers *.Cu *.Mask)
       (net 5 "/3V3") (pinfunction "3V3") (pintype "power_in"))
     (pad "18" thru_hole oval locked (at -2.54 20.32 90) (size 1.7 1.7) (drill 1) (layers *.Cu *.Mask)
-      (net 52 "unconnected-(J10-Pad18)") (pinfunction "GPIO24") (pintype "bidirectional+no_connect"))
+      (net 51 "unconnected-(J10-Pad18)") (pinfunction "GPIO24") (pintype "bidirectional+no_connect"))
     (pad "19" thru_hole oval locked (at 0 22.86 90) (size 1.7 1.7) (drill 1) (layers *.Cu *.Mask)
-      (net 53 "unconnected-(J10-Pad19)") (pinfunction "MOSI0/GPIO10") (pintype "bidirectional+no_connect"))
+      (net 52 "unconnected-(J10-Pad19)") (pinfunction "MOSI0/GPIO10") (pintype "bidirectional+no_connect"))
     (pad "20" thru_hole oval locked (at -2.54 22.86 90) (size 1.7 1.7) (drill 1) (layers *.Cu *.Mask)
       (net 2 "GND") (pinfunction "GND") (pintype "power_in"))
     (pad "21" thru_hole oval locked (at 0 25.4 90) (size 1.7 1.7) (drill 1) (layers *.Cu *.Mask)
-      (net 54 "unconnected-(J10-Pad21)") (pinfunction "MISO0/GPIO9") (pintype "bidirectional+no_connect"))
+      (net 53 "unconnected-(J10-Pad21)") (pinfunction "MISO0/GPIO9") (pintype "bidirectional+no_connect"))
     (pad "22" thru_hole oval locked (at -2.54 25.4 90) (size 1.7 1.7) (drill 1) (layers *.Cu *.Mask)
-      (net 55 "unconnected-(J10-Pad22)") (pinfunction "GPIO25") (pintype "bidirectional+no_connect"))
+      (net 54 "unconnected-(J10-Pad22)") (pinfunction "GPIO25") (pintype "bidirectional+no_connect"))
     (pad "23" thru_hole oval locked (at 0 27.94 90) (size 1.7 1.7) (drill 1) (layers *.Cu *.Mask)
       (net 6 "/SENSOR_SDA") (pinfunction "SCLK0/GPIO11") (pintype "bidirectional"))
@@
       (net 2 "GND") (pinfunction "GND") (pintype "power_in"))
     (pad "26" thru_hole oval locked (at -2.54 30.48 90) (size 1.7 1.7) (drill 1) (layers *.Cu *.Mask)
-      (net 56 "unconnected-(J10-Pad26)") (pinfunction "~{CE1}/GPIO7") (pintype "bidirectional+no_connect"))
+      (net 55 "unconnected-(J10-Pad26)") (pinfunction "~{CE1}/GPIO7") (pintype "bidirectional+no_connect"))
     (pad "27" thru_hole oval locked (at 0 33.02 90) (size 1.7 1.7) (drill 1) (layers *.Cu *.Mask)
       (net 23 "/EEPROM_SDA") (pinfunction "ID_SD/GPIO0") (pintype "bidirectional"))
@@
       (net 24 "/EEPROM_SCL") (pinfunction "ID_SC/GPIO1") (pintype "bidirectional"))
     (pad "29" thru_hole oval locked (at 0 35.56 90) (size 1.7 1.7) (drill 1) (layers *.Cu *.Mask)
-      (net 57 "unconnected-(J10-Pad29)") (pinfunction "GCLK1/GPIO5") (pintype "bidirectional+no_connect"))
+      (net 56 "unconnected-(J10-Pad29)") (pinfunction "GCLK1/GPIO5") (pintype "bidirectional+no_connect"))
     (pad "30" thru_hole oval locked (at -2.54 35.56 90) (size 1.7 1.7) (drill 1) (layers *.Cu *.Mask)
       (net 2 "GND") (pinfunction "GND") (pintype "power_in"))
     (pad "31" thru_hole oval locked (at 0 38.1 90) (size 1.7 1.7) (drill 1) (layers *.Cu *.Mask)
-      (net 58 "unconnected-(J10-Pad31)") (pinfunction "GCLK2/GPIO6") (pintype "bidirectional+no_connect"))
+      (net 57 "unconnected-(J10-Pad31)") (pinfunction "GCLK2/GPIO6") (pintype "bidirectional+no_connect"))
     (pad "32" thru_hole oval locked (at -2.54 38.1 90) (size 1.7 1.7) (drill 1) (layers *.Cu *.Mask)
-      (net 59 "unconnected-(J10-Pad32)") (pinfunction "PWM0/GPIO12") (pintype "bidirectional+no_connect"))
+      (net 58 "unconnected-(J10-Pad32)") (pinfunction "PWM0/GPIO12") (pintype "bidirectional+no_connect"))
     (pad "33" thru_hole oval locked (at 0 40.64 90) (size 1.7 1.7) (drill 1) (layers *.Cu *.Mask)
-      (net 60 "unconnected-(J10-Pad33)") (pinfunction "PWM1/GPIO13") (pintype "bidirectional+no_connect"))
+      (net 59 "unconnected-(J10-Pad33)") (pinfunction "PWM1/GPIO13") (pintype "bidirectional+no_connect"))
     (pad "34" thru_hole oval locked (at -2.54 40.64 90) (size 1.7 1.7) (drill 1) (layers *.Cu *.Mask)
       (net 2 "GND") (pinfunction "GND") (pintype "power_in"))
     (pad "35" thru_hole oval locked (at 0 43.18 90) (size 1.7 1.7) (drill 1) (layers *.Cu *.Mask)
-      (net 61 "unconnected-(J10-Pad35)") (pinfunction "GPIO19/MISO1") (pintype "bidirectional+no_connect"))
+      (net 60 "unconnected-(J10-Pad35)") (pinfunction "GPIO19/MISO1") (pintype "bidirectional+no_connect"))
     (pad "36" thru_hole oval locked (at -2.54 43.18 90) (size 1.7 1.7) (drill 1) (layers *.Cu *.Mask)
-      (net 62 "unconnected-(J10-Pad36)") (pinfunction "GPIO16") (pintype "bidirectional+no_connect"))
+      (net 61 "unconnected-(J10-Pad36)") (pinfunction "GPIO16") (pintype "bidirectional+no_connect"))
     (pad "37" thru_hole oval locked (at 0 45.72 90) (size 1.7 1.7) (drill 1) (layers *.Cu *.Mask)
-      (net 63 "unconnected-(J10-Pad37)") (pinfunction "GPIO26") (pintype "bidirectional+no_connect"))
+      (net 62 "unconnected-(J10-Pad37)") (pinfunction "GPIO26") (pintype "bidirectional+no_connect"))
     (pad "38" thru_hole oval locked (at -2.54 45.72 90) (size 1.7 1.7) (drill 1) (layers *.Cu *.Mask)
-      (net 64 "unconnected-(J10-Pad38)") (pinfunction "GPIO20/MOSI1") (pintype "bidirectional+no_connect"))
+      (net 63 "unconnected-(J10-Pad38)") (pinfunction "GPIO20/MOSI1") (pintype "bidirectional+no_connect"))
     (pad "39" thru_hole oval locked (at 0 48.26 90) (size 1.7 1.7) (drill 1) (layers *.Cu *.Mask)
       (net 2 "GND") (pinfunction "GND") (pintype "power_in"))
     (pad "40" thru_hole oval locked (at -2.54 48.26 90) (size 1.7 1.7) (drill 1) (layers *.Cu *.Mask)
-      (net 65 "unconnected-(J10-Pad40)") (pinfunction "GPIO21/SCLK1") (pintype "bidirectional+no_connect"))
+      (net 64 "unconnected-(J10-Pad40)") (pinfunction "GPIO21/SCLK1") (pintype "bidirectional+no_connect"))
     (model "${KICAD6_3DMODEL_DIR}/Connector_PinSocket_2.54mm.3dshapes/PinSocket_2x20_P2.54mm_Vertical.wrl"
       (offset (xyz 0 0 0))
